File: PSU/PSU/PSU.kicad_pcb (KiCad board)
At the start: 2 copper layers, 99 x 96.5 mm, 25 parts, among them J1 Screw_Terminal_01x03, J2 SW_DIP_x02, J3 Conn_02x08_Odd_Even, J4 Power out, U1 LM7812, U2 LM7912, U3 LM7805_TO220

Commit message: Pyssel
Parts:
- added F1: 1A Polyfuse, Fuse:Fuse_Bourns_MF-RHT200, F.Cu at (85.1, 121.4)
- added F2: 1A Polyfuse, Fuse:Fuse_Bourns_MF-RHT200, F.Cu at (84.9, 115.9)
- added F3: 1A Polyfuse, Fuse:Fuse_Bourns_MF-RHT200, F.Cu at (80.3, 126.0)
- added REF**: MountingHole_2.7mm_M2.5, MountingHole:MountingHole_2.7mm_M2.5, F.Cu at (59.3, 96.1)
- added REF**: MountingHole_2.7mm_M2.5, MountingHole:MountingHole_2.7mm_M2.5, F.Cu at (97.9, 96.5)
- added REF**: MountingHole_2.7mm_M2.5, MountingHole:MountingHole_2.7mm_M2.5, F.Cu at (112.1, 133.3)
- added REF**: MountingHole_2.7mm_M2.5, MountingHole:MountingHole_2.7mm_M2.5, F.Cu at (59.3, 67.4)
- added REF**: MountingHole_2.7mm_M2.5, MountingHole:MountingHole_2.7mm_M2.5, F.Cu at (97.4, 67.6)
- added REF**: MountingHole_2.7mm_M2.5, MountingHole:MountingHole_2.7mm_M2.5, F.Cu at (26.7, 134.4)
- added REF**: MountingHole_2.7mm_M2.5, MountingHole:MountingHole_2.7mm_M2.5, F.Cu at (26.9, 48.3)
- added REF**: MountingHole_2.7mm_M2.5, MountingHole:MountingHole_2.7mm_M2.5, F.Cu at (26.9, 87.8)
- added REF**: MountingHole_2.7mm_M2.5, MountingHole:MountingHole_2.7mm_M2.5, F.Cu at (115.9, 45.7)
- moved J4 5.59 mm to (112.1, 121.4)
Connections:
- C10 pad 1: -12V -> Net-(U2-VO)
- C11 pad 1: +12V -> Net-(D5-A)
- C13 pad 1: +5V -> Net-(D6-A)
- C8 pad 1: +12V -> Net-(D5-A)
- D5 pad 2: +12V -> Net-(D5-A)
- D6 pad 1: +12V -> Net-(D5-A)
- D6 pad 2: +5V -> Net-(D6-A)
- U1 pad 3: +12V -> Net-(D5-A)
- U2 pad 3: -12V -> Net-(U2-VO)
- U3 pad 1: +12V -> Net-(D5-A)
- U3 pad 3: +5V -> Net-(D6-A)
Routing:
- net +12V: track 155.3 -> 31.1 mm
- net Net-(D5-A): track 0.00 -> 92.6 mm
- net +5V: track 90.6 -> 31.2 mm
- net -12V: track 87.9 -> 29.1 mm
- net Net-(D6-A): track 0.00 -> 57.5 mm
- net Net-(U2-VO): track 0.00 -> 29.4 mm
Other:
- board text added: "12V +"
- board text added: "12V -"
- board text added: "5V +"

Commit message: Diverse
Parts:
- U3: value LM7805_TO220 -> LM7805
- moved REF** 4.09 mm to (115.9, 134.8)
- moved REF** 3.78 mm to (24.1, 45.7)
- moved D5 2.79 mm to (33.0, 93.7)
- moved REF** 2.60 mm to (24.1, 134.6)
- moved D6 2.29 mm to (33.0, 114.6)
- moved REF** 1.07 mm to (27.9, 87.8)
Routing:
- net Net-(D5-A): track 92.6 -> 96.7 mm
- net Net-(D6-A): track 57.5 -> 59.8 mm
- net Net-(D1-K): track 157.9 -> 159.5 mm
Other:
- outline, holes or cut-outs redrawn
- board text added: "12V+"
- board text added: "12V-"
- board text added: "5V+"
- board text added: "AC"
- board text added: "AC/Center"
- board text added: "Modular PSU v1.0 Dan Larsson 2024"
- board text added: "PTC Polyfuse 1A"
- board text added: "WayWayWay"
- board text added: "[AC]"
