File: PSU/PSU/PSU.kicad_sch (KiCad schematic)
At the start: 25 parts, among them J1 Screw_Terminal_01x03, J2 SW_DIP_x02, J3 Conn_02x08_Odd_Even, J4 Power out, U1 LM7812, U2 LM7912, U3 LM7805_TO220

Commit message: Pyssel
Parts:
- added F1, F2, F3: 1A Polyfuse, Fuse:Fuse_Bourns_MF-RHT200, symbol Device:Polyfuse
Connections:
- net +12V: now also F1.1; no longer C11.1, C8.1, D5.2 (A), D6.1 (K), U1.3 (VO), U3.1 (VI)
- net +5V: now also F2.1; no longer C13.1, D6.2 (A), U3.3 (VO)
- net -12V: now also F3.2; no longer C10.1, U2.3 (VO)
- new net: C10.1, F3.1, U2.3 (VO)
- new net: C11.1, C8.1, D5.2 (A), D6.1 (K), F1.2, U1.3 (VO), U3.1 (VI)
- new net: C13.1, D6.2 (A), F2.2, U3.3 (VO)
Changed lines of the file:
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@@
   (junction (at 92.71 109.22) (diameter 0) (color 0 0 0 0)
   )
+  (junction (at 187.96 109.22) (diameter 0) (color 0 0 0 0)
+  )
   (junction (at 120.65 109.22) (diameter 0) (color 0 0 0 0)
   )
@@
   )
   (junction (at 81.28 128.27) (diameter 0) (color 0 0 0 0)
-  )
-  (junction (at 187.96 109.22) (diameter 0) (color 0 0 0 0)
   )
   (junction (at 200.66 109.22) (diameter 0) (color 0 0 0 0)
@@
     (stroke (width 0) (type default))
   )
+  (wire (pts (xy 226.06 105.41) (xy 226.06 109.22))
+    (stroke (width 0) (type default))
+  )
   (wire (pts (xy 88.9 132.08) (xy 100.33 132.08))
     (stroke (width 0) (type default))
@@
     (stroke (width 0) (type default))
   )
-  (wire (pts (xy 227.33 97.79) (xy 227.33 109.22))
-    (stroke (width 0) (type default))
-  )
   (wire (pts (xy 156.21 132.08) (xy 161.29 132.08))
     (stroke (width 0) (type default))
@@
     (stroke (width 0) (type default))
   )
+  (wire (pts (xy 189.23 132.08) (xy 189.23 134.62))
+    (stroke (width 0) (type default))
+  )
   (wire (pts (xy 88.9 124.46) (xy 92.71 124.46))
     (stroke (width 0) (type default))
@@
     (stroke (width 0) (type default))
   )
+  (wire (pts (xy 189.23 142.24) (xy 189.23 148.59))
+    (stroke (width 0) (type default))
+  )
   (wire (pts (xy 204.47 97.79) (xy 200.66 97.79))
     (stroke (width 0) (type default))
@@
     (stroke (width 0) (type default))
   )
-  (wire (pts (xy 180.34 132.08) (xy 187.96 132.08))
+  (wire (pts (xy 180.34 132.08) (xy 189.23 132.08))
     (stroke (width 0) (type default))
   )
@@
     (stroke (width 0) (type dash_dot) (color 255 176 22 1))
   )
+  (wire (pts (xy 226.06 92.71) (xy 226.06 97.79))
+    (stroke (width 0) (type default))
+  )
   (wire (pts (xy 203.2 142.24) (xy 207.01 142.24))
     (stroke (width 0) (type default))
@@
   )
   (wire (pts (xy 135.89 116.84) (xy 135.89 119.38))
-    (stroke (width 0) (type default))
-  )
-  (wire (pts (xy 187.96 97.79) (xy 187.96 109.22))
     (stroke (width 0) (type default))
   )
@@
     (stroke (width 0) (type dash_dot) (color 255 176 22 1))
   )
-  (wire (pts (xy 187.96 128.27) (xy 187.96 132.08))
-    (stroke (width 0) (type default))
-  )
   (wire (pts (xy 76.2 109.22) (xy 76.2 119.38))
     (stroke (width 0) (type default))
@@
     (stroke (width 0) (type dash_dot) (color 255 176 22 1))
   )
+  (wire (pts (xy 187.96 105.41) (xy 187.96 109.22))
+    (stroke (width 0) (type default))
+  )
+  (wire (pts (xy 187.96 92.71) (xy 187.96 97.79))
+    (stroke (width 0) (type default))
+  )
   (polyline (pts (xy 124.46 147.32) (xy 102.87 147.32))
     (stroke (width 0) (type dash_dot) (color 255 176 22 1))
@@
     (stroke (width 0) (type dash_dot) (color 255 176 22 1))
   )
-  (wire (pts (xy 219.71 109.22) (xy 227.33 109.22))
+  (wire (pts (xy 219.71 109.22) (xy 226.06 109.22))
     (stroke (width 0) (type default))
   )
@@
     (stroke (width 0) (type dash_dot) (color 255 176 22 1))
   )
+  (wire (pts (xy 187.96 109.22) (xy 195.58 109.22))
+    (stroke (width 0) (type default))
+  )
   (wire (pts (xy 219.71 114.3) (xy 219.71 119.38))
     (stroke (width 0) (type default))
@@
     (stroke (width 0) (type default))
   )
+  (wire (pts (xy 207.01 144.78) (xy 207.01 147.32))
+    (stroke (width 0) (type default))
+  )
   (wire (pts (xy 180.34 109.22) (xy 187.96 109.22))
-    (stroke (width 0) (type default))
-  )
-  (wire (pts (xy 207.01 144.78) (xy 207.01 147.32))
-    (stroke (width 0) (type default))
-  )
-  (wire (pts (xy 187.96 109.22) (xy 195.58 109.22))
     (stroke (width 0) (type default))
   )
@@
     )
   )
-  (symbol (lib_id "power:+12V") (at 187.96 97.79 0) (unit 1)
-    (in_bom yes) (on_board yes) (dnp no) (fields_autoplaced)
-    (property "Reference" "#PWR017" (at 187.96 101.6 0)
-      (effects (font (size 1.27 1.27)) hide)
-    )
-    (property "Value" "+12V" (at 187.96 93.98 0)
+  (symbol (lib_id "power:+12V") (at 187.96 92.71 0) (unit 1)
+    (in_bom yes) (on_board yes) (dnp no) (fields_autoplaced)
+    (property "Reference" "#PWR017" (at 187.96 96.52 0)
+      (effects (font (size 1.27 1.27)) hide)
+    )
+    (property "Value" "+12V" (at 187.96 88.9 0)
       (effects (font (size 1.27 1.27)))
     )
-    (property "Footprint" "" (at 187.96 97.79 0)
-      (effects (font (size 1.27 1.27)) hide)
-    )
-    (property "Datasheet" "" (at 187.96 97.79 0)
+    (property "Footprint" "" (at 187.96 92.71 0)
+      (effects (font (size 1.27 1.27)) hide)
+    )
+    (property "Datasheet" "" (at 187.96 92.71 0)
       (effects (font (size 1.27 1.27)) hide)
     )
@@
         (path "/780e3006-e51c-4736-8f8a-c1e1cf3a82ba"
           (reference "#PWR017") (unit 1)
+        )
+      )
+    )
+  )
+  (symbol (lib_id "Device:Polyfuse") (at 187.96 101.6 0) (unit 1)
+    (in_bom yes) (on_board yes) (dnp no)
+    (property "Reference" "F1" (at 190.5 100.965 0)
+      (effects (font (size 1.27 1.27)) (justify left))
+    )
+    (property "Value" "1A Polyfuse" (at 185.42 105.41 0)
+      (effects (font (size 1.27 1.27)) (justify left))
+    )
+    (property "Footprint" "Fuse:Fuse_Bourns_MF-RHT200" (at 189.23 106.68 0)
+      (effects (font (size 1.27 1.27)) (justify left) hide)
+    )
+    (property "Datasheet" "~" (at 187.96 101.6 0)
+      (effects (font (size 1.27 1.27)) hide)
+    )
+    (pin "1")
+    (pin "2")
+    (instances
+      (project "PSU"
+        (path "/780e3006-e51c-4736-8f8a-c1e1cf3a82ba"
+          (reference "F1") (unit 1)
         )
       )
@@
     )
   )
-  (symbol (lib_id "power:-12V") (at 187.96 128.27 0) (unit 1)
-    (in_bom yes) (on_board yes) (dnp no) (fields_autoplaced)
-    (property "Reference" "#PWR016" (at 187.96 125.73 0)
-      (effects (font (size 1.27 1.27)) hide)
-    )
-    (property "Value" "-12V" (at 187.96 124.46 0)
-      (effects (font (size 1.27 1.27)))
-    )
-    (property "Footprint" "" (at 187.96 128.27 0)
-      (effects (font (size 1.27 1.27)) hide)
-    )
-    (property "Datasheet" "" (at 187.96 128.27 0)
+  (symbol (lib_id "power:-12V") (at 189.23 148.59 180) (unit 1)
+    (in_bom yes) (on_board yes) (dnp no)
+    (property "Reference" "#PWR016" (at 189.23 151.13 0)
+      (effects (font (size 1.27 1.27)) hide)
+    )
+    (property "Value" "-12V" (at 185.42 152.4 0)
+      (effects (font (size 1.27 1.27)) (justify right))
+    )
+    (property "Footprint" "" (at 189.23 148.59 0)
+      (effects (font (size 1.27 1.27)) hide)
+    )
+    (property "Datasheet" "" (at 189.23 148.59 0)
       (effects (font (size 1.27 1.27)) hide)
     )
@@
         (path "/780e3006-e51c-4736-8f8a-c1e1cf3a82ba"
           (reference "#PWR023") (unit 1)
+        )
+      )
+    )
+  )
+  (symbol (lib_id "Device:Polyfuse") (at 189.23 138.43 0) (unit 1)
+    (in_bom yes) (on_board yes) (dnp no)
+    (property "Reference" "F3" (at 191.77 137.795 0)
+      (effects (font (size 1.27 1.27)) (justify left))
+    )
+    (property "Value" "1A Polyfuse" (at 189.23 134.62 0)
+      (effects (font (size 1.27 1.27)) (justify left))
+    )
+    (property "Footprint" "Fuse:Fuse_Bourns_MF-RHT200" (at 190.5 143.51 0)
+      (effects (font (size 1.27 1.27)) (justify left) hide)
+    )
+    (property "Datasheet" "~" (at 189.23 138.43 0)
+      (effects (font (size 1.27 1.27)) hide)
+    )
+    (pin "1")
+    (pin "2")
+    (instances
+      (project "PSU"
+        (path "/780e3006-e51c-4736-8f8a-c1e1cf3a82ba"
+          (reference "F3") (unit 1)
         )
       )
@@
     )
   )
+  (symbol (lib_id "Device:Polyfuse") (at 226.06 101.6 0) (unit 1)
+    (in_bom yes) (on_board yes) (dnp no) (fields_autoplaced)
+    (property "Reference" "F2" (at 228.6 100.965 0)
+      (effects (font (size 1.27 1.27)) (justify left))
+    )
+    (property "Value" "1A Polyfuse" (at 228.6 103.505 0)
+      (effects (font (size 1.27 1.27)) (justify left))
+    )
+    (property "Footprint" "Fuse:Fuse_Bourns_MF-RHT200" (at 227.33 106.68 0)
+      (effects (font (size 1.27 1.27)) (justify left) hide)
+    )
+    (property "Datasheet" "~" (at 226.06 101.6 0)
+      (effects (font (size 1.27 1.27)) hide)
+    )
+    (pin "1")
+    (pin "2")
+    (instances
+      (project "PSU"
+        (path "/780e3006-e51c-4736-8f8a-c1e1cf3a82ba"
+          (reference "F2") (unit 1)
+        )
+      )
+    )
+  )
   (symbol (lib_id "Switch:SW_DIP_x02") (at 63.5 121.92 0) (unit 1)
     (in_bom yes) (on_board yes) (dnp no)
@@
     )
   )
-  (symbol (lib_id "power:+5V") (at 227.33 97.79 0) (unit 1)
-    (in_bom yes) (on_board yes) (dnp no) (fields_autoplaced)
-    (property "Reference" "#PWR018" (at 227.33 101.6 0)
-      (effects (font (size 1.27 1.27)) hide)
-    )
-    (property "Value" "+5V" (at 227.33 93.98 0)
+  (symbol (lib_id "power:+5V") (at 226.06 92.71 0) (unit 1)
+    (in_bom yes) (on_board yes) (dnp no) (fields_autoplaced)
+    (property "Reference" "#PWR018" (at 226.06 96.52 0)
+      (effects (font (size 1.27 1.27)) hide)
+    )
+    (property "Value" "+5V" (at 226.06 88.9 0)
       (effects (font (size 1.27 1.27)))
     )
-    (property "Footprint" "" (at 227.33 97.79 0)
-      (effects (font (size 1.27 1.27)) hide)
-    )
-    (property "Datasheet" "" (at 227.33 97.79 0)
-      (effects (font (size 1.27 1.27)) hide)
-    )
+    (property "Footprint" "" (at 226.06 92.71 0)
+      (effects (font (size 1.27 1.27)) hide)
+    )
+    (property "Datasheet" "" (at 226.06 92.71 0)
+      (effects (font (size 1.27 1.27)) hide)
+    )

Commit message: Diverse
Other:
- note added: "12-15V AC Mount the center tap to Pole 3 None center tapped transformer, use pole 1&3"
- note removed: "12-15V AC Mount the center tap to Pole 1 None center tapped transformer, use pole 1&3"
Changed lines of the file:
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@@
     (effects (font (size 1.27 1.27) (color 255 167 47 1)) (justify left bottom))
   )
-  (text "12-15V AC\n\nMount the center tap to Pole 1\n\nNone center tapped transformer, \nuse pole 1&3"
+  (text "12-15V AC\n\nMount the center tap to Pole 3\n\nNone center tapped transformer, \nuse pole 1&3"
     (at 36.83 110.49 0)
     (effects (font (size 1.27 1.27)) (justify left bottom))
