File: VCO/VCO_1/VCO_1.kicad_sch (KiCad schematic)
At the start: 28 parts, among them J1 Pin3Ring, J2 Pin3Ring, Q1 BC548, Q2 BC558, U1 TL074, U2 40106

Commit message: More work on the VCO
Parts:
- added C?: 1uF, symbol Device:C
- added J? (x3): Pin3Ring, symbol Connector:Barrel_Jack_Switch_Pin3Ring
- added R? (x5): 100K, symbol Device:R
- added R?: 68K, symbol Device:R
- added R? (x2): 1K, symbol Device:R
- added R?: 470K, symbol Device:R
- added R?: 14K, symbol Device:R
- added RV?: 250K, symbol Device:R_Potentiometer
- added RV?: 100K, symbol Device:R_Potentiometer
Connections:
- net +12V: now also RV?.1
- net -12V: now also RV?.3
- net GND: now also J?.1, J?.1, J?.1, R?.1, R?.1, R?.1, R?.1
- net at U1.5 (+): now also U1.10 (+), C?.2, R?.2
- net at U1.6 (-): now also R?.1, R?.2
- net at U1.7: now also R?.1, R?.2
- net at U1.1, U1.2 (-): now also C?.1
- net at U1.12 (+): now also R?.2, R?.2
- net at U1.13 (-): now also U1.14, R?.1
- net at U1.8: now also R?.1
- net at U1.9 (-): now also R?.2, R?.2, R?.2
- new net: J?.3, R?.2 (x2)
- new net: R?.1, RV?.2, RV?.3
- new net: J?.3, RV?.1
- new net: R?.1, RV?.2
Other:
- moved on the sheet: D2, D3, R3, R4, U1A, U1B, U1C, U1D, U1E, U2B, U2C, U2D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
